Commit message: added wheels to the urdf

File: src/archo_description/urdf/archo.urdf.xacro (robot description, xacro)
@@ -5,6 +5,14 @@
     <xacro:property name="base_height" value="0.18"/>
     <xacro:property name="base_mass" value="12.0"/>
+    <xacro:property name="pi" value="3.141592653589793"/>
+    <xacro:property name="wheel_radius" value="0.09"/>
+    <xacro:property name="wheel_width" value="0.04"/>
+    <xacro:property name="wheel_mass" value="0.8"/>
+    <xacro:property name="wheel_y_offset" value="0.20"/>
     <material name="archo_blue">
         <color rgba="0.12 0.35 0.70 1.0"/>
+    </material>
+    <material name="wheel_black">
+        <color rgba="0.0 0.0 0.0 1.0"/>
     </material>
     <link name="base_footprint"/>
@@ -34,4 +42,37 @@
         </inertial>
     </link>
+    <xacro:macro name="drive_wheel" params="prefix y_position">
+        <link name="${prefix}_wheel_link">
+            <visual>
+                <origin xyz="0.0 0.0 0.0" rpy="${pi / 2.0} 0.0 0.0"/>
+                <geometry>
+                    <cylinder radius="${wheel_radius}" length="${wheel_width}"/>
+                </geometry>
+                <material name="wheel_black"/>
+            </visual>
+            <collision>
+                <origin xyz="0.0 0.0 0.0" rpy="${pi / 2.0} 0.0 0.0"/>
+                <geometry>
+                    <cylinder radius="${wheel_radius}" length="${wheel_width}"/>
+                </geometry>
+            </collision>
+            <inertial>
+                <origin xyz="0.0 0.0 0.0" rpy="0.0 0.0 0.0"/>
+                <mass value="${wheel_mass}"/>
+                <inertia
+                    ixx="${wheel_mass * (3*wheel_radius*wheel_radius + wheel_width*wheel_width) / 12.0}"
+                    ixy="0" ixz="0"
+                    iyy="${wheel_mass * wheel_radius * wheel_radius / 2.0}"
+                    iyz="0"
+                    izz="${wheel_mass * (3*wheel_radius*wheel_radius + wheel_width*wheel_width) / 12.0}"/>
+            </inertial>
+        </link>
+        <joint name="${prefix}_wheel_joint" type="continuous">
+            <parent link="base_link"/>
+            <child link="${prefix}_wheel_link"/>
+            <origin xyz="0.0 ${y_position} 0.0" rpy="0.0 0.0 0.0"/>
+            <axis xyz="0.0 1.0 0.0"/>
+        </joint>
+    </xacro:macro>
     <joint name="base_footprint_joint" type="fixed">
         <parent link="base_footprint"/>
@@ -39,3 +80,5 @@
         <origin xyz="0.0 0.0 ${base_height / 2.0}" rpy="0.0 0.0 0.0"/>
     </joint>
+    <xacro:drive_wheel prefix="left" y_position="${wheel_y_offset}"/>
+    <xacro:drive_wheel prefix="right" y_position="${-wheel_y_offset}"/>
 </robot>

Commit message: added an IMU, caster wheel and a LiDAR

File: src/archo_description/urdf/archo.urdf.xacro (robot description, xacro)
@@ -75,4 +75,58 @@
         </joint>
     </xacro:macro>
+    <link name="caster_link">
+        <visual>
+            <geometry>
+                <sphere radius="0.04"/>
+            </geometry>
+        </visual>
+        <collision>
+            <geometry>
+                <sphere radius="0.04"/>
+            </geometry>
+        </collision>
+        <inertial>
+            <mass value="0.15"/>
+            <inertia ixx="0.000096" ixy="0" ixz="0" iyy="0.000096" iyz="0" izz="0.000096"/>
+        </inertial>
+    </link>
+    <link name="laser_link">
+        <visual>
+            <geometry>
+                <cylinder radius="0.045" length="0.04"/>
+            </geometry>
+        </visual>
+        <collision>
+            <geometry>
+                <cylinder radius="0.045" length="0.04"/>
+            </geometry>
+        </collision>
+        <inertial>
+            <mass value="0.2"/>
+            <inertia ixx="0.0002" ixy="0.0" ixz="0.0" iyy="0.0002" iyz="0.0" izz="0.0002"/>
+        </inertial>
+    </link>
+    <link name="imu_link">
+        <visual>
+            <geometry>
+                <box size="0.04 0.03 0.015"/>
+            </geometry>
+        </visual>
+    </link>
+    <joint name="laser_joint" type="fixed">
+        <parent link="base_link"/>
+        <child link="laser_link"/>
+        <origin xyz="0.12 0.0 0.16" rpy="0.0 0.0 0.0"/>
+    </joint>
+    <joint name="imu_joint" type="fixed">
+        <parent link="base_link"/>
+        <child link="imu_link"/>
+        <origin xyz="0.0 0.0 0.11" rpy="0.0 0.0 0.0"/>
+    </joint>
+    <joint name="caster_joint" type="fixed">
+        <parent link="base_link"/>
+        <child link="caster_link"/>
+        <origin xyz="-0.18 0.0 -0.05" rpy="0.0 0.0 0.0"/>
+    </joint>
     <joint name="base_footprint_joint" type="fixed">
         <parent link="base_footprint"/>

Commit message: added essential stuff needed to boot up gazebo sim

File: src/archo_description/urdf/archo.urdf.xacro (robot description, xacro)
@@ -5,5 +5,4 @@
     <xacro:property name="base_height" value="0.18"/>
     <xacro:property name="base_mass" value="12.0"/>
-    <xacro:property name="pi" value="3.141592653589793"/>
     <xacro:property name="wheel_radius" value="0.09"/>
     <xacro:property name="wheel_width" value="0.04"/>
@@ -136,3 +135,23 @@
     <xacro:drive_wheel prefix="left" y_position="${wheel_y_offset}"/>
     <xacro:drive_wheel prefix="right" y_position="${-wheel_y_offset}"/>
+    <ros2_control name="ArchoGazeboSystem" type="system">
+        <hardware>
+            <plugin>gz_ros2_control/GazeboSimSystem</plugin>
+        </hardware>
+        <joint name="left_wheel_joint">
+            <command_interface name="velocity"/>
+            <state_interface name="position"/>
+            <state_interface name="velocity"/>
+        </joint>
+        <joint name="right_wheel_joint">
+            <command_inteface name="velocity"/>
+            <state_interface name="position"/>
+            <state_interface name="velocity"/>
+        </joint>
+    </ros2_control>
+    <gazebo>
+        <plugin filename="gz_ros2_control-system" name="gz_ros2_control::GazeboSimROS2ControlPlugin">
+            <parameters>$(find archo_bringup)/config/controllers.yaml</parameters>
+        </plugin>
+    </gazebo>
 </robot>
